File: Hardware/Qwiic Sound Trigger.brd (EAGLE design)
At the start: 25.4 x 25.4 mm, 74 parts, among them J1 Qwiic Right Angle, J2 PTH, J3 Qwiic Right Angle, Q1 310mA/60V/1.6Ω, U1 VM1010, U2 PCA9536

Commit message: Remove New-Parts
Parts:
- U1: device New_Parts:VM1010 -> SparkFun-Sensors:VM1010
- U2: device New_Parts:MSOP8 -> SparkFun-IC-Conversion:MSOP8
Changed lines of the file:
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@@
 <attribute name="PROD_ID" value="DIO-00819" x="3.81" y="3.175" size="1.778" layer="27" font="vector" ratio="15" rot="R180" display="off"/>
 </element>
-<element name="U2" library="New_Parts" package="MSOP8" value="PCA9536" x="12.7" y="11.938" smashed="yes">
+<element name="U2" library="SparkFun-IC-Conversion" package="MSOP8" value="PCA9536" x="12.7" y="11.938" smashed="yes">
 <attribute name="NAME" x="12.065" y="11.557" size="0.6096" layer="25" font="vector" ratio="20"/>
 <attribute name="PROD_ID" value="IC-15034" x="12.7" y="11.938" size="1.778" layer="27" display="off"/>
@@
 </element>
 <element name="LOGO2" library="SparkFun-Aesthetics" package="ORDERING_INSTRUCTIONS" value="SPECIAL_INSTRUCTIONS-ORDERING" x="34.29" y="50.8" smashed="yes"/>
-<element name="U1" library="New_Parts" package="VM1010" value="VM1010" x="12.7" y="16.51" smashed="yes" rot="R270">
+<element name="U1" library="SparkFun-Sensors" package="VM1010" value="VM1010" x="12.7" y="16.51" smashed="yes" rot="R270">
 <attribute name="DIGIKEY_PART" value="2022-1001-1-ND" x="12.7" y="16.51" size="1.778" layer="27" font="vector" ratio="15" rot="R270" display="off"/>
 <attribute name="MANU_PART" value="VM1010AA" x="12.7" y="16.51" size="1.778" layer="27" font="vector" ratio="15" rot="R270" display="off"/>
