File: Hardware/Qwiic Sound Trigger.sch (EAGLE design)
At the start: 40 parts, among them J1 Qwiic Right Angle, J2 PTH, J3 Qwiic Right Angle, Q1 310mA/60V/1.6Ω, U1 VM1010, U2 PCA9536

Commit message: Remove New-Parts
Parts:
- U1: device New_Parts:VM1010 -> SparkFun-Sensors:VM1010
- U2: device New_Parts:PCA9536 -> SparkFun-IC-Conversion:PCA9536
Changed lines of the file:
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@@
 <part name="D1" library="SparkFun-LED" deviceset="LED-RED" device="0603" value="RED"/>
 <part name="GND3" library="SparkFun-PowerSymbols" deviceset="GND" device=""/>
-<part name="U2" library="New_Parts" deviceset="PCA9536" device=""/>
+<part name="U2" library="SparkFun-IC-Conversion" deviceset="PCA9536" device=""/>
 <part name="SUPPLY11" library="SparkFun-PowerSymbols" deviceset="3.3V" device=""/>
 <part name="GND9" library="SparkFun-PowerSymbols" deviceset="GND" device=""/>
@@
 <part name="LOGO2" library="SparkFun-Aesthetics" deviceset="SPECIAL_INSTRUCTIONS" device="-ORDERING"/>
 <part name="SUPPLY2" library="SparkFun-PowerSymbols" deviceset="3.3V" device=""/>
-<part name="U1" library="New_Parts" deviceset="VM1010" device=""/>
+<part name="U1" library="SparkFun-Sensors" deviceset="VM1010" device=""/>
 <part name="SUPPLY3" library="SparkFun-PowerSymbols" deviceset="3.3V" device=""/>
 <part name="GND1" library="SparkFun-PowerSymbols" deviceset="GND" device=""/>
