File: Hardware/Production/Qwiic Sound Trigger-Panel.brd (EAGLE design)
At the start: 149.1 x 143.3 mm, 1831 parts, among them J1 Qwiic Right Angle, J10 Qwiic Right Angle, J11 PTH, J12 Qwiic Right Angle, J13 Qwiic Right Angle, J14 PTH, J15 Qwiic Right Angle, J16 Qwiic Right Angle, J17 PTH, J18 Qwiic Right Angle, J19 Qwiic Right Angle, J2 PTH, J20 PTH, J21 Qwiic Right Angle, J22 Qwiic Right Angle, J23 PTH, J24 Qwiic Right Angle, J25 Qwiic Right Angle, J26 PTH, J27 Qwiic Right Angle, J28 Qwiic Right Angle, J29 PTH, J3 Qwiic Right Angle, J30 Qwiic Right Angle, J31 Qwiic Right Angle, J32 PTH, J33 Qwiic Right Angle, J34 Qwiic Right Angle, J35 PTH, J36 Qwiic Right Angle, J37 Qwiic Right Angle, J38 PTH, J39 Qwiic Right Angle, J4 Qwiic Right Angle, J40 Qwiic Right Angle, J41 PTH, J42 Qwiic Right Angle, J43 Qwiic Right Angle, J44 PTH, J45 Qwiic Right Angle, J46 Qwiic Right Angle, J47 PTH, J48 Qwiic Right Angle, J49 Qwiic Right Angle, J5 PTH, J50 PTH, J51 Qwiic Right Angle, J52 Qwiic Right Angle, J53 PTH, J54 Qwiic Right Angle, J55 Qwiic Right Angle, J56 PTH, J57 Qwiic Right Angle, J58 Qwiic Right Angle, J59 PTH, J6 Qwiic Right Angle, J60 Qwiic Right Angle, J61 Qwiic Right Angle, J62 PTH, J63 Qwiic Right Angle, J64 Qwiic Right Angle, J65 PTH, J66 Qwiic Right Angle, J67 Qwiic Right Angle, J68 PTH, J69 Qwiic Right Angle, J7 Qwiic Right Angle, J70 Qwiic Right Angle, J71 PTH, J72 Qwiic Right Angle, J73 Qwiic Right Angle, J74 PTH, J75 Qwiic Right Angle, J8 PTH, J9 Qwiic Right Angle, Q1 310mA/60V/1.6Ω, Q10 310mA/60V/1.6Ω, Q11 310mA/60V/1.6Ω, Q12 310mA/60V/1.6Ω, Q13 310mA/60V/1.6Ω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

Commit message: Ready for manufacture
Changed lines of the file:
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@@
 <layer number="128" name="_bValues" color="7" fill="1" visible="no" active="no"/>
 <layer number="129" name="Mask" color="7" fill="1" visible="no" active="no"/>
+<layer number="130" name="SMDSTROOK" color="7" fill="1" visible="no" active="no"/>
 <layer number="131" name="tAdjust" color="7" fill="1" visible="no" active="no"/>
 <layer number="132" name="bAdjust" color="7" fill="1" visible="no" active="no"/>
+<layer number="133" name="bottom_silk" color="7" fill="1" visible="no" active="no"/>
+<layer number="134" name="silk_top" color="7" fill="1" visible="no" active="no"/>
+<layer number="135" name="silk_bottom" color="7" fill="1" visible="no" active="no"/>
+<layer number="136" name="silktop" color="7" fill="1" visible="no" active="no"/>
+<layer number="137" name="silkbottom" color="7" fill="1" visible="no" active="no"/>
+<layer number="138" name="EEE" color="7" fill="1" visible="no" active="no"/>
+<layer number="139" name="_tKeepout" color="7" fill="1" visible="no" active="no"/>
+<layer number="140" name="mbKeepout" color="7" fill="1" visible="no" active="no"/>
+<layer number="141" name="ASSEMBLY_TOP" color="7" fill="1" visible="no" active="no"/>
+<layer number="142" name="mbRestrict" color="7" fill="1" visible="no" active="no"/>
+<layer number="143" name="PLACE_BOUND_TOP" color="7" fill="1" visible="no" active="no"/>
 <layer number="144" name="Drill_legend" color="7" fill="1" visible="no" active="no"/>
+<layer number="145" name="DrillLegend_01-16" color="7" fill="1" visible="no" active="no"/>
+<layer number="146" name="DrillLegend_01-20" color="7" fill="1" visible="no" active="no"/>
+<layer number="147" name="PIN_NUMBER" color="7" fill="1" visible="no" active="no"/>
+<layer number="148" name="DrillLegend_01-20" color="7" fill="1" visible="no" active="no"/>
+<layer number="149" name="DrillLegend_02-15" color="7" fill="1" visible="no" active="no"/>
 <layer number="150" name="Notes" color="7" fill="1" visible="no" active="no"/>
 <layer number="151" name="HeatSink" color="7" fill="1" visible="no" active="no"/>
@@
 <layer number="154" name="FabDoc2" color="7" fill="1" visible="no" active="no"/>
 <layer number="155" name="FabDoc3" color="7" fill="1" visible="no" active="no"/>
+<layer number="166" name="AntennaArea" color="7" fill="1" visible="no" active="no"/>
+<layer number="168" name="4mmHeightArea" color="7" fill="1" visible="no" active="no"/>
+<layer number="191" name="mNets" color="7" fill="1" visible="no" active="no"/>
+<layer number="192" name="mBusses" color="7" fill="1" visible="no" active="no"/>
+<layer number="193" name="mPins" color="7" fill="1" visible="no" active="no"/>
+<layer number="194" name="mSymbols" color="7" fill="1" visible="no" active="no"/>
+<layer number="195" name="mNames" color="7" fill="1" visible="no" active="no"/>
+<layer number="196" name="mValues" color="7" fill="1" visible="no" active="no"/>
 <layer number="199" name="Contour" color="7" fill="1" visible="no" active="no"/>
 <layer number="200" name="200bmp" color="1" fill="10" visible="no" active="no"/>
